Commit message: urdf edit

File: dummy2_gazebo/urdf/base.urdf.xacro (robot description, xacro)
@@ -1,35 +1,43 @@
 <?xml version="1.0"?>
 <robot xmlns:xacro="http://www.ros.org/wiki/xacro" name="dummy2">
-    <xacro:property name="base_width" value="0.40"/>
-    <xacro:property name="base_length" value="0.70"/>
-    <xacro:property name="base_height" value="0.20"/>
-    <xacro:property name="wheel_radius" value="0.14"/>
+    <xacro:property name="base_width" value="0.43"/>
+    <xacro:property name="base_length" value="0.60"/>
+    <xacro:property name="base_height" value="0.10"/>
+    <xacro:property name="wheel_radius" value="0.1"/>
     <xacro:property name="wheel_width" value="0.06"/>
-    <xacro:property name="wheel_ygap" value="0.035"/>
+    <xacro:property name="wheel_ygap" value="0.02"/>
     <xacro:property name="wheel_xoff" value="0.305"/>
-    <xacro:property name="wheel_zoff" value="0.06"/>
+    <xacro:property name="wheel_zoff" value="0.02"/>
+    <xacro:property name="shock_travel" value = "0.09"/>
     <xacro:macro name="box_inertia" params="m w h d">
-        <inertial>
-            <origin xyz="0 0 0" rpy="${pi/2} 0 ${pi/2}"/>
-            <mass value="${m}"/>
-            <inertia ixx="${(m/12)*(h*h + d*d)}" ixy="0.0" ixz="0.0" iyy="${(m/12)*(w*w + d*d)}" iyz="0.0" izz="${(m/12)*(w*w + h*h)}"/>
-        </inertial>
+            <inertia ixx="${(m/12)*(h*h + d*d)}" ixy="0.0" ixz="0.0"
+                     iyy="${(m/12)*(w*w + d*d)}" iyz="0.0"
+                     izz="${(m/12)*(w*w + h*h)}"/>
     </xacro:macro>
     <xacro:macro name="wheel_inertia" params="m r h">
         <inertial>
-            <origin xyz="0 0 0" rpy="${pi/2} 0 0"/>
             <mass value="${m}"/>
-            <inertia ixx="${(m/12) * (3*r*r + h*h)}" ixy="0.0" ixz="0.0" iyy="${(m/12) * (3*r*r + h*h)}" iyz="0.0" izz="${(m/2) * (r*r)}"/>
+            <inertia ixx="${(m/12) * (3*r*r + h*h)}" ixy="0.0" ixz="0.0"
+                     iyy="${(m/12) * (3*r*r + h*h)}" iyz="0.0"
+                     izz="${(m/2) * (r*r)}"/>
         </inertial>
     </xacro:macro>
   <xacro:macro name="sphere_inertia" params="m r">
-    <inertial>
-      <mass value="${m}"/>
-      <inertia ixx="${(2/5) * m * (r*r)}" ixy="0.0" ixz="0.0" iyy="${(2/5) * m * (r*r)}" iyz="0.0" izz="${(2/5) * m * (r*r)}"/>
-    </inertial>
+        <inertial>
+            <mass value="${m}"/>
+            <inertia ixx="${(2/5) * m * (r*r)}" ixy="0.0" ixz="0.0"
+                    iyy="${(2/5) * m * (r*r)}" iyz="0.0"
+                    izz="${(2/5) * m * (r*r)}"/>
+        </inertial>
   </xacro:macro>
-    <link name="base_link">
+    <link name="base_footprint"/>
+    <link name="base_link"/>
+    <joint name="base_joint" type="fixed">
+      <origin xyz="0.0 0.0 0.0" rpy="0.0 0.0 0.0"/>
+      <parent link="base_footprint"/>
+      <child link="base_link"/>
+    </joint>
+    <link name="body_link">
         <visual>
-            <origin xyz="0.0 0.0 -0.05" rpy="0 0 0"/>
             <geometry>
                 <box size="${base_length} ${base_width} ${base_height}"/>
@@ -41,39 +49,112 @@
             </geometry>
         </collision>
-        <xacro:box_inertia m="15.0" w="${base_width}" d="${base_length}" h="${base_height}"/>
-    </link>
-    <link name="base_footprint">
-        <xacro:box_inertia m="0" w="0" h="0" d="0"/>
-    </link>
-    <joint name="base_joint" type="fixed">
-        <origin xyz="0.0 0.0 ${-(wheel_radius+wheel_zoff)}" rpy="0.0 0.0 0.0"/>
+        <inertial>
+          <mass value="2.6"/>
+          <xacro:box_inertia m="2.6" w="${base_width}" d="${base_length}" h="${base_height}"/>
+        </inertial>
+    </link>
+    <joint name="body_joint" type="fixed">
+        <origin xyz="0.0 0.0 ${2*base_height}" rpy="0.0 0.0 0.0"/>
         <parent link="base_link"/>
-        <child link="base_footprint"/>
-    </joint>
-    <xacro:macro name="wheel" params="prefix x_reflect y_reflect">
-    <link name="${prefix}_link">
+        <child link="body_link"/>
+    </joint>
+     <link name="back_left_wheel_link">
+      <xacro:wheel_inertia m="0.1" r="${wheel_radius}" h="${wheel_width}"/>
+      <visual>
+        <geometry>
+          <cylinder length="${wheel_width}" radius="${wheel_radius}"/>
+        </geometry>
+      </visual>
+      <collision>
+        <geometry>
+          <cylinder length="${wheel_width}" radius="${wheel_radius}"/>
+        </geometry>
+      </collision>
+    </link>
+    <link name="back_right_wheel_link">
+      <xacro:wheel_inertia m="0.1" r="${wheel_radius}" h="${wheel_width}"/>
+      <visual>
+        <geometry>
+          <cylinder length="${wheel_width}" radius="${wheel_radius}"/>
+        </geometry>
+      </visual>
+      <collision>
+        <geometry>
+          <cylinder length="${wheel_width}" radius="${wheel_radius}"/>
+        </geometry>
+      </collision>
+    </link>
+    <link name="back_left_wheel_shock">
         <visual>
-            <origin xyz="0.0 0.0 0.0" rpy="${pi/2} 0.0 0.0"/>
-            <geometry>
-                <cylinder radius="${wheel_radius}" length="${wheel_width}"/>
-            </geometry>
-        </visual>
-        <collision>
-            <origin xyz="0.0 0.0 0.0" rpy="${pi/2} 0.0 0.0"/>
-            <geometry>
-                <cylinder radius="${wheel_radius}" length="${wheel_width}"/>
-            </geometry>
-        </collision>
-        <xacro:wheel_inertia m="0.5" r="${wheel_radius}" h="${wheel_width}"/>
-    </link>
-    <joint name="${prefix}_joint" type="continuous">
-        <origin xyz="${x_reflect*wheel_xoff} ${y_reflect*(base_width/2+wheel_ygap)} ${-wheel_zoff}" rpy="0.0 0.0 0.0"/>
-        <parent link="base_link"/>
-        <child link="${prefix}_link"/>
-        <axis xyz="0.0 1.0 0.0"/>
-    </joint>
-    </xacro:macro>
-    <xacro:wheel prefix="drivewhl_l" x_reflect="-1" y_reflect="1"/>
-    <xacro:wheel prefix="drivewhl_r" x_reflect="-1" y_reflect="-1"/>
+        <origin xyz="0 0 0.1" rpy="0 0 0"/>
+        <geometry>
+          <cylinder length="0.05" radius="0.01"/>
+        </geometry>
+        <material name="silver">
+          <color rgba="0.75 0.75 0.75 1"/>
+        </material>
+      </visual>
+      <collision>
+        <origin xyz="0 0 0.1" rpy="0 0 0"/>
+        <geometry>
+          <cylinder length="0.05" radius="0.01"/>
+        </geometry>
+      </collision>
+      <inertial>
+        <mass value="0.01"/>
+        <inertia ixx="0.015" iyy="0.0375" izz="0.0375"
+                ixy="0" ixz="0" iyz="0"/>
+      </inertial>
+    </link>
+    <link name="back_right_wheel_shock">
+        <visual>
+        <origin xyz="0 0 0.1" rpy="0 0 0"/>
+        <geometry>
+          <cylinder length="0.05" radius="0.01"/>
+        </geometry>
+        <material name="silver">
+          <color rgba="0.75 0.75 0.75 1"/>
+        </material>
+      </visual>
+      <collision>
+        <origin xyz="0 0 0.1" rpy="0 0 0"/>
+        <geometry>
+          <cylinder length="0.05" radius="0.01"/>
+        </geometry>
+      </collision>
+      <inertial>
+        <mass value="0.01"/>
+        <inertia ixx="0.015" iyy="0.0375" izz="0.0375"
+                ixy="0" ixz="0" iyz="0"/>
+      </inertial>
+    </link>
+    <joint name="back_left_shock_joint" type="prismatic">
+      <origin xyz="${-wheel_xoff} ${(base_width/2)} ${shock_travel}" rpy="0.0 0.0 0.0"/>
+      <parent link="base_link"/>
+      <child link="back_left_wheel_shock"/>
+      <axis xyz="0 0 1"/>
+      <limit lower="0" upper="${shock_travel}" effort="100" velocity="100"/>
+    </joint>
+    <joint name="back_left_wheel_joint" type="continuous">
+      <origin xyz="0.0 0.0 0.0" rpy="${-pi/2} 0.0 0.0"/>
+      <parent link="back_left_wheel_shock"/>
+      <child link="back_left_wheel_link"/>
+      <axis xyz="0 0 1"/>
+      <limit effort="10000" velocity="500"/>
+    </joint>
+    <joint name="back_right_shock_joint" type="prismatic">
+      <origin xyz="${-wheel_xoff} ${-(base_width/2)} ${shock_travel}" rpy="0.0 0.0 0.0"/>
+      <parent link="base_link"/>
+      <child link="back_right_wheel_shock"/>
+      <axis xyz="0 0 1"/>
+      <limit lower="0" upper="${shock_travel}" effort="100" velocity="100"/>
+    </joint>
+    <joint name="back_right_wheel_joint" type="continuous">
+      <origin xyz="0.0 0.0 0.0" rpy="${-pi/2} 0.0 0.0"/>
+      <parent link="back_right_wheel_shock"/>
+      <child link="back_right_wheel_link"/>
+      <axis xyz="0 0 1"/>
+      <limit effort="10000" velocity="500"/>
+    </joint>
     <link name="front_left_wheel_steer">
       <visual>
@@ -93,5 +174,5 @@
         <mass value="0.1"/>
         <inertia ixx="5.1458e-5" iyy="5.1458e-5" izz="6.125e-5"
-                ixy="0" ixz="0" iyz="0"/>
+                 ixy="0" ixz="0" iyz="0"/>
       </inertial>
     </link>
@@ -107,8 +188,8 @@
         </geometry>
       </collision>
-      <xacro:wheel_inertia m="0.5" r="${wheel_radius}" h="${wheel_width}"/>
-    </link>
-    <!-- <link name="front_left_wheel_shock">
-        <visual>
+      <xacro:wheel_inertia m="0.1" r="${wheel_radius}" h="${wheel_width}"/>
+    </link>
+    <link name="front_left_wheel_shock">
+      <visual>
         <origin xyz="0 0 0.1" rpy="0 0 0"/>
         <geometry>
@@ -130,16 +211,16 @@
                 ixy="0" ixz="0" iyz="0"/>
       </inertial>
-    </link> -->
-    <!-- <joint name="front_left_shock_joint" type="prismatic">
-      <limit lower="0" upper="0.09" effort="100" velocity="100"/>
+    </link>
+    <joint name="front_left_shock_joint" type="prismatic">
+      <limit lower="0" upper="${shock_travel}" effort="100" velocity="100"/>
       <axis xyz="0 0 1"/>
       <parent link="base_link"/>
       <child link="front_left_wheel_shock"/>
-      <origin rpy="0 0 0" xyz="${wheel_xoff} ${(base_width/2+wheel_ygap)} ${-(wheel_zoff)}"/>
-    </joint> -->
+      <origin rpy="0 0 0" xyz="${wheel_xoff} ${(base_width/2)} ${shock_travel}"/>
+    </joint>
     <joint name="front_left_wheel_steer_joint" type="revolute">
       <limit lower="-1" upper="1" effort="1" velocity="5"/>
       <axis xyz="0 0 1"/>
-      <parent link="base_link"/>
+      <parent link="front_left_wheel_shock"/>
       <child link="front_left_wheel_steer"/>
       <origin rpy="0 0 0" xyz="0 0 0"/>
@@ -149,5 +230,5 @@
       <parent link="front_left_wheel_steer"/>
       <child link="front_left_wheel"/>
-      <origin rpy="${-pi/2} 0 0" xyz="${wheel_xoff} ${(base_width/2+wheel_ygap)} ${-1*(wheel_zoff)}"/>
+      <origin rpy="${-pi/2} 0 0" xyz="0 0 0"/>
     </joint>
     <link name="front_right_wheel_steer">
@@ -182,7 +263,7 @@
         </geometry>
       </collision>
-      <xacro:wheel_inertia m="0.5" r="${wheel_radius}" h="${wheel_width}"/>
-    </link>
-    <!-- <link name="front_right_wheel_shock">
+      <xacro:wheel_inertia m="0.1" r="${wheel_radius}" h="${wheel_width}"/>
+    </link>
+    <link name="front_right_wheel_shock">
       <visual>
       <origin xyz="0 0 0.1" rpt="0 0 0"/>
@@ -204,124 +285,28 @@
     </link>
     <joint name="front_right_shock_joint" type="prismatic">
-      <limit lower="0.0" upper="0.09" effort="100" velocity="100"/>
+      <limit lower="0.0" upper="${shock_travel}" effort="100" velocity="100"/>
       <axis xyz="0.0 0.0 1.0"/>
       <parent link="base_link"/>
       <child link="front_right_wheel_shock"/>
-      <origin rpy="0 0 0" xyz="${wheel_xoff} ${-(base_width/2+wheel_ygap)} ${-(wheel_zoff)}"/>
-    </joint> -->
+      <origin rpy="0 0 0" xyz="${wheel_xoff} ${-(base_width/2)} ${shock_travel}"/>
+    </joint>
     <joint name="front_right_wheel_steer_joint" type="revolute">
       <limit lower="-1" upper="1" effort="1" velocity="5"/>
       <axis xyz="0.0 0.0 1.0"/>
-      <parent link="base_link"/>
+      <parent link="front_right_wheel_shock"/>
       <child link="front_right_wheel_steer"/>
       <origin xyz="0.0 0.0 0.0" rpy="0.0 0.0 0.0"/>
     </joint>
     <joint name="front_right_wheel_joint" type="continuous">
-      <axis xyz="1.0 0.0 1.0"/>
+      <axis xyz="0 0.0 1.0"/>
       <parent link="front_right_wheel_steer"/>
       <child link="front_right_wheel"/>
-      <origin rpy="${-pi/2} 0.0 0.0" xyz="${wheel_xoff} ${-1*(base_width/2+wheel_ygap)} ${-1*(wheel_zoff)}"/>
-    </joint>
-    <link name="imu_link">
-    <visual>
-      <geometry>
-        <box size="0.1 0.1 0.1"/>
-      </geometry>
-    </visual>
-    <collision>
-      <geometry>
-        <box size="0.1 0.1 0.1"/>
-      </geometry>
-    </collision>
-    <xacro:box_inertia m="0.1" w="0.1" d="0.1" h="0.1"/>
-  </link>
-  <joint name="imu_joint" type="fixed">
-    <parent link="base_link"/>
-    <child link="imu_link"/>
-    <origin xyz="0 0 0.01"/>
-  </joint>
-  <gazebo reference="imu_link">
-    <gravity>true</gravity>
-    <sensor name="twr_imu" type="imu">
-      <always_on>true</always_on>
-      <update_rate>100</update_rate>
-      <visualize>true</visualize>
-      <imu>
-        <orientation>
-          <x>
-            <noise type="gaussian">
-              <mean>0.0</mean>
-              <stddev>2e-3</stddev>
-            </noise>
-          </x>
-          <y>
-            <noise type="gaussian">
-              <mean>0.0</mean>
-              <stddev>2e-3</stddev>
-            </noise>
-          </y>
-          <z>
-            <noise type="gaussian">
-              <mean>0.0</mean>
-              <stddev>2e-3</stddev>
-            </noise>
-          </z>
-        </orientation>
-        <angular_velocity>
-          <x>
-            <noise type="gaussian">
-              <mean>0.0</mean>
-              <stddev>2e-4</stddev>
-            </noise>
-          </x>
-          <y>
-            <noise type="gaussian">
-              <mean>0.0</mean>
-              <stddev>2e-4</stddev>
-            </noise>
-          </y>
-          <z>
-            <noise type="gaussian">
-              <mean>0.0</mean>
-              <stddev>2e-4</stddev>
-            </noise>
-          </z>
-        </angular_velocity>
-        <linear_acceleration>
-          <x>
-            <noise type="gaussian">
-              <mean>0.0</mean>
-              <stddev>1.7e-2</stddev>
-            </noise>
-          </x>
-          <y>
-            <noise type="gaussian">
-              <mean>0.0</mean>
-              <stddev>1.7e-2</stddev>
-            </noise>
-          </y>
-          <z>
-            <noise type="gaussian">
-              <mean>0.0</mean>
-              <stddev>1.7e-2</stddev>
-            </noise>
-          </z>
-        </linear_acceleration>
-      </imu>
-      <plugin name="two_wheeled_robot_imu" filename="libgazebo_ros_imu_sensor.so">
-        <initial_orientation_as_reference>false</initial_orientation_as_reference>
-        <frame_name>imu_link</frame_name>
-        <ros>
-          <namespace>/imu</namespace>
-          <remapping>~/out:=data</remapping>
-        </ros>
-      </plugin>
-    </sensor>
-</gazebo>
- <link name="lidar_link">
+      <origin rpy="${-pi/2} 0.0 0.0" xyz="0 0 0"/>
+    </joint>
+  <link name="lidar_link">
     <inertial>
       <origin xyz="0 0 0" rpy="0 0 0"/>
-      <mass value="2.0"/>
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